File: KiCad files/Tranzistorski_pretvarač.kicad_pcb (KiCad board)
At the start: 2 copper layers, 99.9 x 92.6 mm, 32 parts, among them J1 Screw_Terminal_01x01, J2 Screw_Terminal_01x01, J3 Conn_01x03_Male, J4 Conn_01x01_Male, J5 Screw_Terminal_01x01, J6 Conn_01x01_Male, J7 Conn_01x01_Male, J8 Conn_01x01_Male, J9 Screw_Terminal_01x01, Q1 IRLZ44N, U1 SG3524

Commit message: update
Other:
- board text added: "github"
- board text removed: "Dokumentacija:"
Changed lines of the file:
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@@
   (gr_line (start 188.749817 145.2) (end 188.749266 59.6) (layer "Edge.Cuts") (width 0.1))
   (gr_line (start 185.249817 148.7) (end 92.150184 148.7) (layer "Edge.Cuts") (width 0.1))
-  (gr_text "Dokumentacija:" (at 142.2 61) (layer "B.SilkS")
+  (gr_text "github" (at 142.2 61) (layer "B.SilkS")
     (effects (font (size 2 2) (thickness 0.5)) (justify mirror))
   )
@@
   (dimension (type aligned) (layer "User.9")
     (pts (xy 188.75 150.9) (xy 88.8 150.9))
-    (height -10.6)
-    (gr_text "99,9500 mm" (at 138.775 160.35) (layer "User.9")
-      (effects (font (size 1 1) (thickness 0.15)))
+    (height -5.2)
+    (gr_text "99,9500 mm" (at 138.775 153.8) (layer "User.9")
+      (effects (font (size 2 2) (thickness 0.3)))
     )
     (format (units 3) (units_format 1) (precision 4))
@@
   (dimension (type aligned) (layer "User.9")
     (pts (xy 185.249266 56.1) (xy 185.249817 148.7))
-    (height -12)
-    (gr_text "92,6000 mm" (at 199.549541 102.399915 270.0003403) (layer "User.9")
+    (height -7.950183)
+    (gr_text "92,6000 mm" (at 195.499724 102.399939 270.0003403) (layer "User.9")
       (effects (font (size 2 2) (thickness 0.3)))
     )

Commit message: update
Parts:
- moved J4 22.5 mm to (121.8, 139.5)
- moved J6 10.4 mm to (143.9, 139.5)
- moved J7 10.1 mm to (132.9, 139.5)
Connections:
- J4 pad 1: Net-(D2-Pad2) -> Net-(J4-Pad1)
- RV1 pad 2: Net-(RV1-Pad2) -> Net-(J4-Pad1)
- U1 pad 2: Net-(RV1-Pad2) -> Net-(J4-Pad1)
Routing:
- net Net-(J4-Pad1): track 0.00 -> 87.6 mm
- net Net-(RV1-Pad2): track 35.7 -> 0.00 mm
- net Net-(D2-Pad2): track 44.0 -> 14.9 mm
- net Net-(J6-Pad1): track 78.4 -> 71.5 mm
Other:
- board text added: "POT"
Changed lines of the file:
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@@
   (net 13 "unconnected-(U1-Pad4)")
   (net 14 "unconnected-(U1-Pad5)")
-  (net 15 "Net-(RV1-Pad2)")
+  (net 15 "Net-(J4-Pad1)")
   (net 16 "Net-(Q1-Pad1)")
   (net 17 "Net-(J6-Pad1)")
@@
       (net 9 "Net-(R2-Pad2)") (pinfunction "1") (pintype "passive"))
     (pad "2" thru_hole oval (at 0 7 270) (size 2 3) (drill 1) (layers *.Cu *.Mask)
-      (net 15 "Net-(RV1-Pad2)") (pinfunction "2") (pintype "passive"))
+      (net 15 "Net-(J4-Pad1)") (pinfunction "2") (pintype "passive"))
     (pad "3" thru_hole oval (at 2.5 7 270) (size 2 3) (drill 1) (layers *.Cu *.Mask)
       (net 8 "Net-(R1-Pad1)") (pinfunction "3") (pintype "passive"))
@@
   )
   (footprint "footprint:oscil" (layer "F.Cu")
-    (at 133.533333 139.53)
+    (at 143.933332 139.53)
     (descr "Through hole straight pin header, 1x02, 2.54mm pitch, single row")
     (tags "Through hole pin header THT 1x02 2.54mm single row")
@@
   )
   (footprint "footprint:oscil" (layer "F.Cu")
-    (at 144.266666 139.53)
+    (at 121.8 139.53)
     (descr "Through hole straight pin header, 1x02, 2.54mm pitch, single row")
     (tags "Through hole pin header THT 1x02 2.54mm single row")
@@
     (fp_line (start 1.8 -1.8) (end -1.8 -1.8) (layer "F.CrtYd") (width 0.05))
     (pad "1" thru_hole circle (at 0 0) (size 1.7 1.7) (drill 1) (layers *.Cu *.Mask)
-      (net 6 "Net-(D2-Pad2)") (pinfunction "Pin_1") (pintype "passive"))
+      (net 15 "Net-(J4-Pad1)") (pinfunction "Pin_1") (pintype "passive"))
     (pad "1" thru_hole oval (at 0 2.54) (size 1.7 1.7) (drill 1) (layers *.Cu *.Mask)
-      (net 6 "Net-(D2-Pad2)") (pinfunction "Pin_1") (pintype "passive"))
+      (net 15 "Net-(J4-Pad1)") (pinfunction "Pin_1") (pintype "passive"))
     (model "${MOJ3D}/usica.STEP"
       (offset (xyz 0 -1.27 -2.5))
@@
   )
   (footprint "footprint:oscil" (layer "F.Cu")
-    (at 122.8 139.53)
+    (at 132.866666 139.53)
     (descr "Through hole straight pin header, 1x02, 2.54mm pitch, single row")
     (tags "Through hole pin header THT 1x02 2.54mm single row")
@@
       (net 4 "Net-(C4-Pad1)") (pinfunction "INV._INPUT") (pintype "passive"))
     (pad "2" thru_hole oval locked (at 0 2.54) (size 2.4 1.6) (drill 0.8) (layers *.Cu *.Mask)
-      (net 15 "Net-(RV1-Pad2)") (pinfunction "NON_INV._INPUT") (pintype "passive"))
+      (net 15 "Net-(J4-Pad1)") (pinfunction "NON_INV._INPUT") (pintype "passive"))
     (pad "3" thru_hole oval locked (at 0 5.08) (size 2.4 1.6) (drill 0.8) (layers *.Cu *.Mask)
       (net 12 "unconnected-(U1-Pad3)") (pinfunction "OSC./SYNC.") (pintype "passive+no_connect"))
@@
     (effects (font (size 3 3) (thickness 0.5)))
   )
-  (gr_text "OUT" (at 144.5 145.6) (layer "F.SilkS")
+  (gr_text "POT" (at 121.8 145.7) (layer "F.SilkS")
     (effects (font (size 1.5 1.5) (thickness 0.3)))
   )
@@
     (effects (font (size 1.5 1.5) (thickness 0.3)))
   )
-  (gr_text "CT" (at 122.8 145.6) (layer "F.SilkS")
+  (gr_text "CT" (at 132.9 145.6) (layer "F.SilkS")
     (effects (font (size 1.5 1.5) (thickness 0.3)))
   )
-  (gr_text "COL" (at 133.5 145.6) (layer "F.SilkS")
+  (gr_text "COL" (at 144 145.6) (layer "F.SilkS")
     (effects (font (size 1.5 1.5) (thickness 0.3)))
   )
@@
   (segment (start 133.8 71.4) (end 129.104733 66.704733) (width 2) (layer "F.Cu") (net 5))
   (segment (start 133.8 86.02) (end 133.8 71.4) (width 2) (layer "F.Cu") (net 5))
-  (segment (start 168.85 134.75) (end 149.046666 134.75) (width 1.27) (layer "F.Cu") (net 6))
-  (segment (start 149.046666 134.75) (end 144.266666 139.53) (width 1.27) (layer "F.Cu") (net 6))
-  (segment (start 144.266666 139.53) (end 144.266666 142.07) (width 1.27) (layer "F.Cu") (net 6))
   (segment (start 158.96 95.1) (end 158.96 109.99) (width 1.27) (layer "B.Cu") (net 6))
-  (segment (start 122.8 142.07) (end 122.8 139.53) (width 1.27) (layer "F.Cu") (net 7))
   (segment (start 130.2 125.7) (end 130.2 118.135) (width 1.27) (layer "F.Cu") (net 7))
   (segment (start 120.943 98.76) (end 118.64 98.76) (width 1.27) (layer "F.Cu") (net 7))
-  (segment (start 130.2 125.7) (end 122.8 133.1) (width 1.27) (layer "F.Cu") (net 7))
+  (segment (start 135.3 137.096666) (end 132.866666 139.53) (width 1.27) (layer "F.Cu") (net 7))
+  (segment (start 135.3 130.8) (end 135.3 137.096666) (width 1.27) (layer "F.Cu") (net 7))
   (segment (start 118.64 98.76) (end 117.2 100.2) (width 1.27) (layer "F.Cu") (net 7))
   (segment (start 130.185 115.585) (end 130.185 118.12) (width 1.27) (layer "F.Cu") (net 7))
   (segment (start 117.2 110.6) (end 120 113.4) (width 1.27) (layer "F.Cu") (net 7))
+  (segment (start 132.866666 142.07) (end 132.866666 139.53) (width 1.27) (layer "F.Cu") (net 7))
+  (segment (start 130.2 125.7) (end 135.3 130.8) (width 1.27) (layer "F.Cu") (net 7))
   (segment (start 120 113.4) (end 128 113.4) (width 1.27) (layer "F.Cu") (net 7))
   (segment (start 130.2 118.135) (end 130.185 118.12) (width 1.27) (layer "F.Cu") (net 7))
   (segment (start 128 113.4) (end 130.185 115.585) (width 1.27) (layer "F.Cu") (net 7))
   (segment (start 117.2 100.2) (end 117.2 110.6) (width 1.27) (layer "F.Cu") (net 7))
-  (segment (start 122.8 133.1) (end 122.8 139.53) (width 1.27) (layer "F.Cu") (net 7))
   (segment (start 96.42 105.6305) (end 95.6895 104.9) (width 1.27) (layer "F.Cu") (net 8))
   (segment (start 96.42 117.4) (end 96.42 105.6305) (width 1.27) (layer "F.Cu") (net 8))
@@
   (segment (start 113.4 98.92) (end 116.1 96.22) (width 1.27) (layer "F.Cu") (net 10))
   (segment (start 116.1 96.22) (end 120.943 96.22) (width 1.27) (layer "F.Cu") (net 10))
-  (segment (start 105.6 102.4) (end 108.6 99.4) (width 1.27) (layer "F.Cu") (net 15))
-  (segment (start 108.6 99.4) (end 108.6 93.1) (width 1.27) (layer "F.Cu") (net 15))
-  (segment (start 95.6895 102.4) (end 105.6 102.4) (width 1.27) (layer "F.Cu") (net 15))
   (segment (start 120.943 86.06) (end 115.64 86.06) (width 1.27) (layer "F.Cu") (net 15))
+  (segment (start 108.3 102.4) (end 108.6 102.1) (width 1.27) (layer "F.Cu") (net 15))
   (segment (start 115.64 86.06) (end 108.6 93.1) (width 1.27) (layer "F.Cu") (net 15))
+  (segment (start 115.5 133.23) (end 121.8 139.53) (width 1.27) (layer "F.Cu") (net 15))
+  (segment (start 108.6 100.7) (end 106.9 102.4) (width 1.27) (layer "F.Cu") (net 15))
+  (segment (start 115.5 119) (end 115.5 133.23) (width 1.27) (layer "F.Cu") (net 15))
+  (segment (start 106.9 102.4) (end 106.8 102.4) (width 1.27) (layer "F.Cu") (net 15))
+  (segment (start 121.8 142.07) (end 121.8 139.53) (width 1.27) (layer "F.Cu") (net 15))
+  (segment (start 106.8 102.4) (end 108.3 102.4) (width 1.27) (layer "F.Cu") (net 15))
+  (segment (start 108.6 102.1) (end 108.6 104.1) (width 1.27) (layer "F.Cu") (net 15))
+  (segment (start 108.6 104.1) (end 108.6 112.1) (width 1.27) (layer "F.Cu") (net 15))
+  (segment (start 108.6 93.1) (end 108.6 100.7) (width 1.27) (layer "F.Cu") (net 15))
+  (segment (start 106.9 102.4) (end 108.6 104.1) (width 1.27) (layer "F.Cu") (net 15))
+  (segment (start 95.6895 102.4) (end 106.8 102.4) (width 1.27) (layer "F.Cu") (net 15))
+  (segment (start 108.6 112.1) (end 115.5 119) (width 1.27) (layer "F.Cu") (net 15))
+  (segment (start 108.6 100.7) (end 108.6 102.1) (width 1.27) (layer "F.Cu") (net 15))
   (segment (start 141.48 98.92) (end 141.58 98.92) (width 1.27) (layer "B.Cu") (net 16))
   (segment (start 161.5 95.1) (end 161.5 92.9) (width 1.27) (layer "B.Cu") (net 16))
@@
   (segment (start 134.08 96.08) (end 133.8 95.8) (width 1.27) (layer "F.Cu") (net 17))
   (segment (start 139.6 109.08) (end 137.72 109.08) (width 1.27) (layer "F.Cu") (net 17))
-  (segment (start 133.533333 142.07) (end 133.533333 139.53) (width 1.27) (layer "F.Cu") (net 17))
-  (segment (start 133.533333 139.53) (end 137.863333 135.2) (width 1.27) (layer "F.Cu") (net 17))
-  (segment (start 142.2 135.2) (end 144 133.4) (width 1.27) (layer "F.Cu") (net 17))
-  (segment (start 144 133.4) (end 144 122.6) (width 1.27) (layer "F.Cu") (net 17))
+  (segment (start 143.933332 142.07) (end 143.933332 122.666668) (width 1.27) (layer "F.Cu") (net 17))
   (segment (start 137.72 108.92) (end 136.7 107.9) (width 1.27) (layer "F.Cu") (net 17))
   (segment (start 136.7 110.1) (end 136.7 110.6) (width 1.27) (layer "F.Cu") (net 17))
@@
   (segment (start 136.7 101.82) (end 133.8 98.92) (width 1.27) (layer "F.Cu") (net 17))
   (segment (start 128.563 93.68) (end 131.68 93.68) (width 1.27) (layer "F.Cu") (net 17))
-  (segment (start 144 122.6) (end 136.7 115.3) (width 1.27) (layer "F.Cu") (net 17))
   (segment (start 133.8 95.8) (end 133.8 98.92) (width 1.27) (layer "F.Cu") (net 17))
   (segment (start 128.563 91.14) (end 128.563 93.68) (width 1.27) (layer "F.Cu") (net 17))
-  (segment (start 136.7 115.3) (end 136.7 110.6) (width 1.27) (layer "F.Cu") (net 17))
   (segment (start 131.68 93.68) (end 133.8 95.8) (width 1.27) (layer "F.Cu") (net 17))
-  (segment (start 137.863333 135.2) (end 142.2 135.2) (width 1.27) (layer "F.Cu") (net 17))
+  (segment (start 136.7 115.433336) (end 136.7 110.6) (width 1.27) (layer "F.Cu") (net 17))
+  (segment (start 143.933332 122.666668) (end 136.7 115.433336) (width 1.27) (layer "F.Cu") (net 17))
   (segment (start 139.6 96.08) (end 134.08 96.08) (width 1.27) (layer "F.Cu") (net 17))
   (segment (start 136.7 107.9) (end 136.7 101.82) (width 1.27) (layer "F.Cu") (net 17))

Commit message: update
Parts:
- renumbered J1 to B1, J2 to B2, J5 to B3, J9 to B4, J4 to J1, J7 to J2, J6 to J3, J8 to J4, J3 to J5
Connections:
- net Net-(J4-Pad1) renamed /POT
- net Net-(J6-Pad1) renamed /COL
Other:
- board text removed: "github"

Commit message: final
Parts:
- removed the G*** at (149.4, 67.1)
- added G***: LOGO, footprint:tvz2, F.Cu at (149.2, 62.6)
