File: KiCad files/Tranzistorski_pretvarač.kicad_sch (KiCad schematic)
At the start: 31 parts, among them J1 Screw_Terminal_01x01, J2 Screw_Terminal_01x01, J3 Conn_01x03_Male, J4 Conn_01x01_Male, J5 Screw_Terminal_01x01, J6 Conn_01x01_Male, J7 Conn_01x01_Male, J8 Conn_01x01_Male, J9 Screw_Terminal_01x01, Q1 IRLZ44N, U1 SG3524, U2 PC817

Commit message: test
Parts:
- removed R5: 2k, Resistor_THT:R_Axial_DIN0207_L6.3mm_D2.5mm_P10.16mm_Horizontal, symbol Device:R_Small
- removed U2: PC817, Package_DIP:DIP-4_W7.62mm, symbol Isolator:PC817
- R1: value 1k -> 2k7
- R2: value 3k -> 2k7
- R4: value 10k -> 4k7
Connections:
- net at J6.1 (Pin_1), R4.2, U1.12 (COLLECTOR_A)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: now also R6.1, R7.2
Other:
- note added: "- C1-4 obavezno kvalitetni blok kondenzatori, ne elektroliti - footprint potenciometra nema one dvije rupe - dodati qr kod kao link na dokumentaciju - invertirati signal? - nazivi priključnica - nazivi mjernih mjesta - keepout area oko vijka mosfeta - testirati v1 na induktivnom trošilu - da li treba onaj desni GND? - dodati tvz logo - smanjti svoj logo - manji elektrolit? Da li on uopće treba? -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"
- note removed: "- pogledati na osciloskopu izlaz mosfeta - C1-4 obavezno kvalitetni blok kondenzatori, ne elektroliti - footprint potenciometra nema one dvije rupe - dodati qr kod kao link na dokumentaciju - invertirati signal? - nazivi priključnica - nazivi mjernih mjesta - keepout area oko vijka mosfeta - testirati v1 na induktivnom trošilu - da li treba onaj desni GND? - dodati tvz logo - smanjti svoj logo - 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"
- moved on the sheet: D2, J4, J5, J6, J9, Q1, R4, R6, R7

Commit message: test
Parts:
- R7: value 220 -> 330
Changed lines of the file:
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@@
       (effects (font (size 1.27 1.27)) (justify left))
     )
-    (property "Value" "220" (id 1) (at 140.97 71.12 90)
+    (property "Value" "330" (id 1) (at 140.97 71.12 90)
       (effects (font (size 1 1)) (justify left))
     )
@@
     )
     (path "/175ff781-f4ed-43bd-a280-c6060ba3a4b7"
-      (reference "R7") (unit 1) (value "220") (footprint "Resistor_THT:R_Axial_DIN0207_L6.3mm_D2.5mm_P10.16mm_Horizontal")
+      (reference "R7") (unit 1) (value "330") (footprint "Resistor_THT:R_Axial_DIN0207_L6.3mm_D2.5mm_P10.16mm_Horizontal")
     )
     (path "/aaa37d05-6fec-40cb-a150-9cdb3d2105a5"

Commit message: update
Parts:
- C5: footprint Capacitor_THT:CP_Radial_D13.0mm_P5.00mm -> Capacitor_THT:CP_Radial_D17.0mm_P7.50mm
Changed lines of the file:
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@@
       (effects (font (size 1.27 1.27)) (justify left))
     )
-    (property "Footprint" "Capacitor_THT:CP_Radial_D13.0mm_P5.00mm" (id 2) (at 121.92 47.625 0)
+    (property "Footprint" "Capacitor_THT:CP_Radial_D17.0mm_P7.50mm" (id 2) (at 121.92 47.625 0)
       (effects (font (size 1.27 1.27)) hide)
     )
@@
     )
     (path "/c39275c1-7838-4ebf-8487-0dfef76f3fff"
-      (reference "C5") (unit 1) (value "1000u") (footprint "Capacitor_THT:CP_Radial_D13.0mm_P5.00mm")
+      (reference "C5") (unit 1) (value "1000u") (footprint "Capacitor_THT:CP_Radial_D17.0mm_P7.50mm")
     )
     (path "/28c0ef69-12df-44c9-8574-1b20346ebf0f"

Commit message: qr code
Other:
- note added: "- C1-4 obavezno kvalitetni blok kondenzatori, ne elektroliti"
- note removed: "- C1-4 obavezno kvalitetni blok kondenzatori, ne elektroliti - footprint potenciometra nema one dvije rupe - dodati qr kod kao link na dokumentaciju - invertirati signal? - nazivi priključnica - nazivi mjernih mjesta - keepout area oko vijka mosfeta - testirati v1 na induktivnom trošilu - da li treba onaj desni GND? - dodati tvz logo - smanjti svoj logo - manji elektrolit? Da li on uopće treba? -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"
Changed lines of the file:
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@@
     (effects (font (size 3 3) (thickness 0.6) bold) (justify left bottom))
   )
-  (text "- C1-4 obavezno kvalitetni blok kondenzatori, ne elektroliti\n- footprint potenciometra nema one dvije rupe\n- dodati qr kod kao link na dokumentaciju\n- invertirati signal?\n- nazivi priključnica\n- nazivi mjernih mjesta\n- keepout area oko vijka mosfeta\n- testirati v1 na induktivnom trošilu\n- da li treba onaj desni GND?\n- dodati tvz logo\n- smanjti svoj logo\n- manji elektrolit? Da li on uopće treba?\n- na footprintu J9 staviti plavu ili zelenu pruključnicu\n- potenciometar rupe\n- koje sve napone je potrebno mjeriti?"
-    (at 19.05 195.58 0)
+  (text "- C1-4 obavezno kvalitetni blok kondenzatori, ne elektroliti"
+    (at 18.415 188.595 0)
     (effects (font (size 1.27 1.27)) (justify left bottom))
   )

Commit message: update
Other:
- moved on the sheet: H1, H2, H3, H4, J1, J2

Commit message: update
Connections:
- net at D2.2 (A), J9.1 (Pin_1), Q1.2 (D): no longer J4.1 (Pin_1)
- net at RV1.2, U1.2 (NON_INV._INPUT): now also J4.1 (Pin_1)
Other:
- moved on the sheet: J4, J5, J7, J9
Changed lines of the file:
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@@
   (junction (at 124.46 86.36) (diameter 0) (color 0 0 0 0)
+  )
+  (junction (at 56.515 63.5) (diameter 0) (color 0 0 0 0)
   )
   (junction (at 125.73 71.12) (diameter 0) (color 0 0 0 0)
@@
     (stroke (width 0) (type default) (color 0 0 0 0))
   )
-  (wire (pts (xy 166.37 53.34) (xy 171.45 53.34))
-    (stroke (width 0) (type default) (color 0 0 0 0))
-  )
   (wire (pts (xy 124.46 86.36) (xy 124.46 91.44))
     (stroke (width 0) (type default) (color 0 0 0 0))
@@
     (stroke (width 0) (type default) (color 0 0 0 0))
   )
-  (wire (pts (xy 166.37 55.88) (xy 166.37 60.96))
-    (stroke (width 0) (type default) (color 0 0 0 0))
-  )
   (wire (pts (xy 81.28 86.36) (xy 76.2 86.36))
     (stroke (width 0) (type default) (color 0 0 0 0))
@@
     (stroke (width 0) (type default) (color 0 0 0 0))
   )
-  (wire (pts (xy 152.4 60.96) (xy 154.94 60.96))
-    (stroke (width 0) (type default) (color 0 0 0 0))
-  )
-  (wire (pts (xy 53.34 63.5) (xy 81.28 63.5))
+  (wire (pts (xy 53.34 63.5) (xy 56.515 63.5))
     (stroke (width 0) (type default) (color 0 0 0 0))
   )
@@
     (stroke (width 0) (type default) (color 0 0 0 0))
   )
-  (wire (pts (xy 171.45 55.88) (xy 166.37 55.88))
-    (stroke (width 0) (type default) (color 0 0 0 0))
-  )
   (wire (pts (xy 55.245 127) (xy 55.245 129.54))
     (stroke (width 0) (type default) (color 0 0 0 0))
@@
     (stroke (width 0) (type default) (color 0 0 0 0))
   )
+  (wire (pts (xy 56.515 63.5) (xy 81.28 63.5))
+    (stroke (width 0) (type default) (color 0 0 0 0))
+  )
   (wire (pts (xy 57.15 91.44) (xy 64.77 91.44))
     (stroke (width 0) (type default) (color 0 0 0 0))
   )
-  (wire (pts (xy 68.58 83.82) (xy 68.58 86.36))
-    (stroke (width 0) (type default) (color 0 0 0 0))
-  )
   (polyline (pts (xy 78.74 118.745) (xy 78.74 147.955))
     (stroke (width 0) (type default) (color 0 0 0 0))
@@
     (stroke (width 0) (type default) (color 0 0 0 0))
   )
-  (wire (pts (xy 166.37 50.8) (xy 166.37 53.34))
-    (stroke (width 0) (type default) (color 0 0 0 0))
-  )
   (wire (pts (xy 57.15 60.96) (xy 62.23 60.96))
     (stroke (width 0) (type default) (color 0 0 0 0))
@@
     (stroke (width 0) (type default) (color 0 0 0 0))
   )
-  (wire (pts (xy 166.37 60.96) (xy 154.94 60.96))
+  (wire (pts (xy 154.94 60.96) (xy 171.45 60.96))
     (stroke (width 0) (type default) (color 0 0 0 0))
   )
@@
     (stroke (width 0) (type default) (color 0 0 0 0))
   )
+  (wire (pts (xy 56.515 63.5) (xy 56.515 66.04))
+    (stroke (width 0) (type default) (color 0 0 0 0))
+  )
   (wire (pts (xy 137.16 71.12) (xy 137.16 73.66))
     (stroke (width 0) (type default) (color 0 0 0 0))
   )
-  (wire (pts (xy 154.94 50.8) (xy 166.37 50.8))
+  (wire (pts (xy 154.94 50.8) (xy 171.45 50.8))
     (stroke (width 0) (type default) (color 0 0 0 0))
   )
@@
     )
   )
-  (symbol (lib_id "Connector:Conn_01x01_Male") (at 68.58 91.44 90) (unit 1)
-    (in_bom yes) (on_board yes)
-    (property "Reference" "J7" (id 0) (at 69.85 88.9 90)
+  (symbol (lib_id "Connector:Conn_01x01_Male") (at 63.5 83.82 0) (unit 1)
+    (in_bom yes) (on_board yes)
+    (property "Reference" "J7" (id 0) (at 66.04 85.09 0)
       (effects (font (size 1.27 1.27)) (justify right))
     )
-    (property "Value" "Conn_01x01_Male" (id 1) (at 69.4182 92.6716 90)
+    (property "Value" "Conn_01x01_Male" (id 1) (at 62.2684 84.6582 90)
       (effects (font (size 1.27 1.27)) (justify right) hide)
     )
-    (property "Footprint" "footprint:oscil" (id 2) (at 68.58 91.44 0)
-      (effects (font (size 1.27 1.27)) hide)
-    )
-    (property "Datasheet" "~" (id 3) (at 68.58 91.44 0)
-      (effects (font (size 1.27 1.27)) hide)
-    )
-    (pin "1")
-  )
-  (symbol (lib_id "Connector:Conn_01x01_Male") (at 147.32 60.96 0) (unit 1)
-    (in_bom yes) (on_board yes)
-    (property "Reference" "J4" (id 0) (at 149.86 62.23 0)
+    (property "Footprint" "footprint:oscil" (id 2) (at 63.5 83.82 0)
+      (effects (font (size 1.27 1.27)) hide)
+    )
+    (property "Datasheet" "~" (id 3) (at 63.5 83.82 0)
+      (effects (font (size 1.27 1.27)) hide)
+    )
+    (pin "1")
+  )
+  (symbol (lib_id "Connector:Conn_01x01_Male") (at 56.515 71.12 90) (unit 1)
+    (in_bom yes) (on_board yes)
+    (property "Reference" "J4" (id 0) (at 57.785 68.58 0)
       (effects (font (size 1.27 1.27)) (justify right))
     )
-    (property "Value" "Conn_01x01_Male" (id 1) (at 146.0884 61.7982 90)
+    (property "Value" "Conn_01x01_Male" (id 1) (at 57.3532 72.3516 90)
       (effects (font (size 1.27 1.27)) (justify right) hide)
     )
-    (property "Footprint" "footprint:oscil" (id 2) (at 147.32 60.96 0)
-      (effects (font (size 1.27 1.27)) hide)
-    )
-    (property "Datasheet" "~" (id 3) (at 147.32 60.96 0)
+    (property "Footprint" "footprint:oscil" (id 2) (at 56.515 71.12 0)
+      (effects (font (size 1.27 1.27)) hide)
+    )
+    (property "Datasheet" "~" (id 3) (at 56.515 71.12 0)
       (effects (font (size 1.27 1.27)) hide)
     )
@@
     (pin "1")
   )
-  (symbol (lib_id "Connector:Screw_Terminal_01x01") (at 176.53 55.88 0) (unit 1)
-    (in_bom yes) (on_board yes) (fields_autoplaced)
-    (property "Reference" "J9" (id 0) (at 178.562 56.359 0)
-      (effects (font (size 1.27 1.27)) (justify left))
-    )
-    (property "Value" "Screw_Terminal_01x01" (id 1) (at 178.562 57.7466 0)
+  (symbol (lib_id "Connector:Screw_Terminal_01x01") (at 176.53 60.96 0) (unit 1)
+    (in_bom yes) (on_board yes)
+    (property "Reference" "J9" (id 0) (at 178.435 60.96 0)
+      (effects (font (size 1.27 1.27)) (justify left))
+    )
+    (property "Value" "Screw_Terminal_01x01" (id 1) (at 178.562 62.8266 0)
       (effects (font (size 1.27 1.27)) (justify left) hide)
     )
-    (property "Footprint" "footprint:DELTRON 4mm banana socket - black" (id 2) (at 176.53 55.88 0)
-      (effects (font (size 1.27 1.27)) hide)
-    )
-    (property "Datasheet" "~" (id 3) (at 176.53 55.88 0)
+    (property "Footprint" "footprint:DELTRON 4mm banana socket - black" (id 2) (at 176.53 60.96 0)
+      (effects (font (size 1.27 1.27)) hide)
+    )
+    (property "Datasheet" "~" (id 3) (at 176.53 60.96 0)
       (effects (font (size 1.27 1.27)) hide)
     )
@@
     (pin "2")
   )
-  (symbol (lib_id "Connector:Screw_Terminal_01x01") (at 176.53 53.34 0) (unit 1)
-    (in_bom yes) (on_board yes) (fields_autoplaced)
-    (property "Reference" "J5" (id 0) (at 178.562 53.819 0)
-      (effects (font (size 1.27 1.27)) (justify left))
-    )
-    (property "Value" "Screw_Terminal_01x01" (id 1) (at 178.562 55.2066 0)
+  (symbol (lib_id "Connector:Screw_Terminal_01x01") (at 176.53 50.8 0) (unit 1)
+    (in_bom yes) (on_board yes)
+    (property "Reference" "J5" (id 0) (at 178.435 50.8 0)
+      (effects (font (size 1.27 1.27)) (justify left))
+    )
+    (property "Value" "Screw_Terminal_01x01" (id 1) (at 178.562 52.6666 0)
       (effects (font (size 1.27 1.27)) (justify left) hide)
     )
-    (property "Footprint" "footprint:DELTRON 4mm banana socket - red" (id 2) (at 176.53 53.34 0)
-      (effects (font (size 1.27 1.27)) hide)
-    )
-    (property "Datasheet" "~" (id 3) (at 176.53 53.34 0)
-      (effects (font (size 1.27 1.27)) hide)
-    )
+    (property "Footprint" "footprint:DELTRON 4mm banana socket - red" (id 2) (at 176.53 50.8 0)
+      (effects (font (size 1.27 1.27)) hide)
+    )
+    (property "Datasheet" "~" (id 3) (at 176.53 50.8 0)
+      (effects (font (size 1.27 1.27)) hide)
+    )

Commit message: update
Parts:
- renumbered J1 to B1, J2 to B2, J5 to B3, J9 to B4, J4 to J1, J7 to J2, J6 to J3, J8 to J4, J3 to J5
Connections:
- net COL: now reaches J3.1 (Pin_1), R4.2, R6.1, R7.2, U1.12 (COLLECTOR_A), U1.13 (COLLECTOR_B)
- net POT: now reaches J1.1 (Pin_1), RV1.2, U1.2 (NON_INV._INPUT)
Other:
- note added: "IZLAZ"
- note removed: "CHOPPER"
- moved on the sheet: B1, B2, B3, B4, C1, C2, C3, C4, C5, C6, D2, H1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

Commit message: update
Other:
- note removed: "- C1-4 obavezno kvalitetni blok kondenzatori, ne elektroliti"
Changed lines of the file:
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@@
     (effects (font (size 3 3) (thickness 0.6) bold) (justify left bottom))
-  )
-  (text "- C1-4 obavezno kvalitetni blok kondenzatori, ne elektroliti"
-    (at 18.415 188.595 0)
-    (effects (font (size 1.27 1.27)) (justify left bottom))
   )
   (label "COL" (at 165.1 86.995 0)
