File: KiCad files/Tranzistorski_pretvarač.kicad_sch (KiCad schematic)
At the start: 29 parts, among them J1 Conn_01x01_Male, J2 Conn_01x01_Male, J3 Conn_01x01_Male, J4 Conn_01x01_Male, J5 Conn_01x03_Male, Q1 IRLZ44N, U1 SG3524

Commit message: update
Parts:
- R1, R2: value 2k7 -> (none)
Changed lines of the file:
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@@
       (effects (font (size 1.27 1.27)) (justify left))
     )
-    (property "Value" "2k7" (id 1) (at 106.045 76.835 90)
+    (property "Value" "" (id 1) (at 106.045 76.835 90)
       (effects (font (size 0.8 0.8)) (justify left))
     )
@@
       (effects (font (size 1.27 1.27)) (justify left))
     )
-    (property "Value" "2k7" (id 1) (at 93.345 88.265 90)
+    (property "Value" "" (id 1) (at 93.345 88.265 90)
       (effects (font (size 1 1)) (justify left))
     )
@@
     )
     (path "/9885de07-c0e2-46ed-99b0-19922238a1da"
-      (reference "R1") (unit 1) (value "2k7") (footprint "Resistor_THT:R_Axial_DIN0207_L6.3mm_D2.5mm_P10.16mm_Horizontal")
+      (reference "R1") (unit 1) (value "3k3") (footprint "Resistor_THT:R_Axial_DIN0207_L6.3mm_D2.5mm_P10.16mm_Horizontal")
     )
     (path "/7ef843e3-5636-4e38-9ebf-4b485d9a70ad"
-      (reference "R2") (unit 1) (value "2k7") (footprint "Resistor_THT:R_Axial_DIN0207_L6.3mm_D2.5mm_P10.16mm_Horizontal")
+      (reference "R2") (unit 1) (value "4k7") (footprint "Resistor_THT:R_Axial_DIN0207_L6.3mm_D2.5mm_P10.16mm_Horizontal")
     )
     (path "/c4a3f633-b32e-46ee-bfce-e27e9e1e700b"

Commit message: v2rev2
Parts:
- R1: value (none) -> 3k3
- R2: value (none) -> 4k7
Other:
- moved on the sheet: B1, B2, B3, B4, C1, C2, C3, C4, C5, C6, D2, H1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

Commit message: update
Parts:
- C1: value 470n -> (none)
- C2, C3: value 1u -> (none)
- R3: value 10k -> (none)
Other:
- note added: "RT (R_{3}) = ${c4a3f633-b32e-46ee-bfce-e27e9e1e700b:VALUE} C_{1} = ${b0c859f5-da41-47d1-bec8-2ebfb3c59348:VALUE} C_{2} = ${bc9eb4d6-7e31-48fd-9445-439387c6ebca:VALUE} C_{3} = ${9fb25102-befc-44c7-8668-d9e721c05423:VALUE} ________________ f = 1.3/RT*C bez jumpera: f_{1} = 1.3/RT*C_{2} = 1.3/2.2*0.47 = 1257 Hz jumper lijevo: f_{2} = 1.3/RT*(C_{1}||C_{2}) = 1.3/2.2*(1+0.47) = 401 Hz jumper desno: f_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"
Changed lines of the file:
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@@
     (effects (font (size 3 3) (thickness 0.6) bold) (justify left bottom))
+  )
+  (text "RT (R_{3}) = ${c4a3f633-b32e-46ee-bfce-e27e9e1e700b:VALUE}\nC_{1} = ${b0c859f5-da41-47d1-bec8-2ebfb3c59348:VALUE}\nC_{2} = ${bc9eb4d6-7e31-48fd-9445-439387c6ebca:VALUE}\nC_{3} = ${9fb25102-befc-44c7-8668-d9e721c05423:VALUE}\n________________\n\nf = 1.3/RT*C\n\nbez jumpera:	f_{1} = 1.3/RT*C_{2} = 1.3/2.2*0.47 = 1257 Hz\n\njumper lijevo:	f_{2} = 1.3/RT*(C_{1}||C_{2}) = 1.3/2.2*(1+0.47) = 401 Hz\n\njumper desno:	f_{3} = 1.3/RT*(C_{2}||C_{3}) = 1.3/2.2*(0.47+0.22) = 856 Hz\n"
+    (at 17.78 186.055 0)
+    (effects (font (size 2.54 2.54)) (justify left bottom))
   )
   (label "COL" (at 164.465 72.39 0)
@@
   (symbol (lib_id "Device:C_Small") (at 101.6 105.41 0) (unit 1)
     (in_bom yes) (on_board yes) (fields_autoplaced)
-    (property "Reference" "C3" (id 0) (at 103.9241 104.5078 0)
-      (effects (font (size 1.27 1.27)) (justify left))
-    )
-    (property "Value" "1u" (id 1) (at 103.9241 107.2829 0)
+    (property "Reference" "C3" (id 0) (at 103.9241 104.5816 0)
+      (effects (font (size 1.27 1.27)) (justify left))
+    )
+    (property "Value" "" (id 1) (at 103.9241 107.1185 0)
       (effects (font (size 1.27 1.27)) (justify left))
     )
@@
   (symbol (lib_id "Device:C_Small") (at 81.28 105.41 0) (unit 1)
     (in_bom yes) (on_board yes) (fields_autoplaced)
-    (property "Reference" "C1" (id 0) (at 83.6041 104.5078 0)
-      (effects (font (size 1.27 1.27)) (justify left))
-    )
-    (property "Value" "470n" (id 1) (at 83.6041 107.2829 0)
+    (property "Reference" "C1" (id 0) (at 83.6041 104.5816 0)
+      (effects (font (size 1.27 1.27)) (justify left))
+    )
+    (property "Value" "" (id 1) (at 83.6041 107.1185 0)
       (effects (font (size 1.27 1.27)) (justify left))
     )
@@
   (symbol (lib_id "Device:C_Small") (at 91.44 105.41 0) (unit 1)
     (in_bom yes) (on_board yes) (fields_autoplaced)
-    (property "Reference" "C2" (id 0) (at 93.7641 104.5078 0)
-      (effects (font (size 1.27 1.27)) (justify left))
-    )
-    (property "Value" "1u" (id 1) (at 93.7641 107.2829 0)
+    (property "Reference" "C2" (id 0) (at 93.7641 104.5816 0)
+      (effects (font (size 1.27 1.27)) (justify left))
+    )
+    (property "Value" "" (id 1) (at 93.7641 107.1185 0)
       (effects (font (size 1.27 1.27)) (justify left))
     )
@@
       (effects (font (size 1.27 1.27)) (justify left))
     )
-    (property "Value" "10k" (id 1) (at 118.11 92.71 90)
+    (property "Value" "" (id 1) (at 118.11 92.71 90)
       (effects (font (size 1 1)) (justify left))
     )
@@
     )
     (path "/b0c859f5-da41-47d1-bec8-2ebfb3c59348"
-      (reference "C1") (unit 1) (value "470n") (footprint "Capacitor_THT:C_Rect_L7.2mm_W2.5mm_P5.00mm_FKS2_FKP2_MKS2_MKP2")
+      (reference "C1") (unit 1) (value "1uF") (footprint "Capacitor_THT:C_Rect_L7.2mm_W2.5mm_P5.00mm_FKS2_FKP2_MKS2_MKP2")
     )
     (path "/bc9eb4d6-7e31-48fd-9445-439387c6ebca"
-      (reference "C2") (unit 1) (value "1u") (footprint "Capacitor_THT:C_Rect_L7.2mm_W2.5mm_P5.00mm_FKS2_FKP2_MKS2_MKP2")
+      (reference "C2") (unit 1) (value "0.47uF") (footprint "Capacitor_THT:C_Rect_L7.2mm_W2.5mm_P5.00mm_FKS2_FKP2_MKS2_MKP2")
     )
     (path "/9fb25102-befc-44c7-8668-d9e721c05423"
-      (reference "C3") (unit 1) (value "1u") (footprint "Capacitor_THT:C_Rect_L7.2mm_W2.5mm_P5.00mm_FKS2_FKP2_MKS2_MKP2")
+      (reference "C3") (unit 1) (value "0.22uF") (footprint "Capacitor_THT:C_Rect_L7.2mm_W2.5mm_P5.00mm_FKS2_FKP2_MKS2_MKP2")
     )
     (path "/a370ec26-8275-468a-aa41-9aca758bd6c2"
@@
     )
     (path "/c4a3f633-b32e-46ee-bfce-e27e9e1e700b"
-      (reference "R3") (unit 1) (value "10k") (footprint "Resistor_THT:R_Axial_DIN0207_L6.3mm_D2.5mm_P10.16mm_Horizontal")
+      (reference "R3") (unit 1) (value "2k2") (footprint "Resistor_THT:R_Axial_DIN0207_L6.3mm_D2.5mm_P10.16mm_Horizontal")
     )
     (path "/05858591-8f32-4847-89b2-2700c2978cb5"

Commit message: Update Tranzistorski_pretvarač.kicad_sch
Parts:
- C1: value (none) -> 1uF
- C2: value (none) -> 0.47uF
- C3: value (none) -> 0.22uF
- Q1: value IRLZ44N -> (none)
- R3: value (none) -> 2k2
Other:
- note added: "- zamijeniti IRLZ44N sa IRFZ44N jer ima viši napon Ugs (20V umjesto 16V)"
Changed lines of the file:
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@@
     (effects (font (size 2.54 2.54)) (justify left bottom))
+  )
+  (text "- zamijeniti IRLZ44N sa IRFZ44N jer ima viši napon Ugs (20V umjesto 16V)"
+    (at 24.13 24.13 0)
+    (effects (font (size 3 3)) (justify left bottom))
   )
   (label "COL" (at 164.465 72.39 0)
@@
   (symbol (lib_id "Transistor_FET:IRLZ44N") (at 194.31 72.39 0) (unit 1)
     (in_bom yes) (on_board yes) (fields_autoplaced)
-    (property "Reference" "Q1" (id 0) (at 199.517 71.4815 0)
-      (effects (font (size 1.27 1.27)) (justify left))
-    )
-    (property "Value" "IRLZ44N" (id 1) (at 199.517 74.2566 0)
+    (property "Reference" "Q1" (id 0) (at 199.517 71.5553 0)
+      (effects (font (size 1.27 1.27)) (justify left))
+    )
+    (property "Value" "" (id 1) (at 199.517 74.0922 0)
       (effects (font (size 1.27 1.27)) (justify left))
     )
@@
       (effects (font (size 1.27 1.27)) (justify left))
     )
-    (property "Value" "" (id 1) (at 103.9241 107.1185 0)
+    (property "Value" "0.22uF" (id 1) (at 103.9241 107.1185 0)
       (effects (font (size 1.27 1.27)) (justify left))
     )
@@
       (effects (font (size 1.27 1.27)) (justify left))
     )
-    (property "Value" "" (id 1) (at 83.6041 107.1185 0)
+    (property "Value" "1uF" (id 1) (at 83.6041 107.1185 0)
       (effects (font (size 1.27 1.27)) (justify left))
     )
@@
       (effects (font (size 1.27 1.27)) (justify left))
     )
-    (property "Value" "" (id 1) (at 93.7641 107.1185 0)
+    (property "Value" "0.47uF" (id 1) (at 93.7641 107.1185 0)
       (effects (font (size 1.27 1.27)) (justify left))
     )
@@
       (effects (font (size 1.27 1.27)) (justify left))
     )
-    (property "Value" "" (id 1) (at 118.11 92.71 90)
+    (property "Value" "2k2" (id 1) (at 118.11 92.71 90)
       (effects (font (size 1 1)) (justify left))
     )
@@
     )
     (path "/40bb1208-0574-4b9c-8a7f-a1fbec81c789"
-      (reference "Q1") (unit 1) (value "IRLZ44N") (footprint "footprint:TO-220F-3_Horizontal_TabDown")
+      (reference "Q1") (unit 1) (value "IRFZ44N") (footprint "footprint:TO-220F-3_Horizontal_TabDown")
     )
     (path "/9885de07-c0e2-46ed-99b0-19922238a1da"

Commit message: generate documentation
Parts:
- Q1: value (none) -> IRFZ44N
Changed lines of the file:
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@@
       (effects (font (size 1.27 1.27)) (justify left))
     )
-    (property "Value" "" (id 1) (at 199.517 74.0922 0)
+    (property "Value" "IRFZ44N" (id 1) (at 199.517 74.0922 0)
       (effects (font (size 1.27 1.27)) (justify left))
     )
